Commit message: added arm part description

File: src/robot_description/urdf/robot_description.urdf.xacro (robot description, xacro)
@@ -1,4 +1,5 @@
 <?xml version="1.0"?>
 <robot name="four_wheel_robot" xmlns:xacro="http://www.ros.org/wiki/xacro">
+    <!-- mobile robot properties -->
     <xacro:property name="base_length" value="0.6"/>
     <xacro:property name="base_width" value="0.4"/>
@@ -11,4 +12,16 @@
     <xacro:property name="wheel_y_offset" value="0.225"/>
     <xacro:property name="wheel_z_offset" value="-0.05"/>
+    <!-- arm robot properties -->
+     <xacro:property name="link_radius" value="0.025"/>
+    <xacro:property name="shoulder_length" value="0.05"/>
+    <xacro:property name="upper_arm_length" value="0.15"/>
+    <xacro:property name="forearm_length" value="0.15"/>
+    <xacro:property name="wrist_length" value="0.06"/>
+    <xacro:property name="gripper_length" value="0.05"/>
+    <xacro:property name="finger_length" value="0.04"/>
+    <!-- gripper properties -->
+     <xacro:property name="finger_width" value="0.015"/>
+    <xacro:property name="finger_thickness" value="0.01"/>
+    <xacro:property name="finger_gap" value="0.015"/>
     <link name="base_footprint"/>
     <link name="base_link">
@@ -91,3 +104,130 @@
         <origin xyz="0.1 0 ${base_height/2}" rpy="0 0 0"/>
     </joint>
+    <link name="arm_base_link">
+        <visual>
+            <geometry>
+                <cylinder radius="${link_radius*1.5}" length="${shoulder_length}"/>
+            </geometry>
+            <material name="arm_color">
+                <color rgba="0.8 0.3 0.1 1.0"/>
+            </material>
+        </visual>
+    </link>
+    <joint name="arm_base_joint" type="fixed">
+        <parent link="arm_mount_link"/>
+        <child link="arm_base_link"/>
+        <origin xyz="0 0 ${shoulder_length/2}" rpy="0 0 0"/>
+    </joint>
+    <link name="shoulder_link">
+        <visual>
+            <geometry>
+                <cylinder radius="${link_radius}" length="${shoulder_length}"/>
+            </geometry>
+            <material name="arm_color"/>
+        </visual>
+    </link>
+    <joint name="shoulder_yaw_joint" type="revolute">
+        <parent link="arm_base_link"/>
+        <child link="shoulder_link"/>
+        <origin xyz="0 0 ${shoulder_length/2}" rpy="0 0 0"/>
+        <axis xyz="0 0 1"/>
+        <limit lower="-3.1416" upper="3.1416" effort="10" velocity="1.0"/>
+    </joint>
+    <link name="upper_arm_link">
+        <visual>
+            <origin xyz="0 0 ${upper_arm_length/2}" rpy="0 0 0"/>
+            <geometry>
+                <cylinder radius="${link_radius}" length="${upper_arm_length}"/>
+            </geometry>
+            <material name="arm_color"/>
+        </visual>
+    </link>
+    <joint name="shoulder_pitch_joint" type="revolute">
+        <parent link="shoulder_link"/>
+        <child link="upper_arm_link"/>
+        <origin xyz="0 0 ${shoulder_length/2}" rpy="0 0 0"/>
+        <axis xyz="0 1 0"/>
+        <limit lower="-1.5708" upper="1.5708" effort="10" velocity="1.0"/>
+    </joint>
+    <link name="forearm_link">
+        <visual>
+            <origin xyz="0 0 ${forearm_length/2}" rpy="0 0 0"/>
+            <geometry>
+                <cylinder radius="${link_radius*0.8}" length="${forearm_length}"/>
+            </geometry>
+            <material name="arm_color"/>
+        </visual>
+    </link>
+    <joint name="elbow_pitch_joint" type="revolute">
+        <parent link="upper_arm_link"/>
+        <child link="forearm_link"/>
+        <origin xyz="0 0 ${upper_arm_length}" rpy="0 0 0"/>
+        <axis xyz="0 1 0"/>
+        <limit lower="0" upper="2.618" effort="10" velocity="1.0"/>
+    </joint>
+    <link name="wrist_link">
+        <visual>
+            <origin xyz="0 0 ${wrist_length/2}" rpy="0 0 0"/>
+            <geometry>
+                <cylinder radius="${link_radius*0.7}" length="${wrist_length}"/>
+            </geometry>
+            <material name="arm_color"/>
+        </visual>
+    </link>
+    <joint name="wrist_pitch_joint" type="revolute">
+        <parent link="forearm_link"/>
+        <child link="wrist_link"/>
+        <origin xyz="0 0 ${forearm_length}" rpy="0 0 0"/>
+        <axis xyz="0 1 0"/>
+        <limit lower="-1.5708" upper="1.5708" effort="5" velocity="1.0"/>
+    </joint>
+    <link name="gripper_base_link">
+        <visual>
+            <origin xyz="0 0 ${gripper_length/2}" rpy="0 0 0"/>
+            <geometry>
+                <box size="0.05 0.06 ${gripper_length}"/>
+            </geometry>
+            <material name="gripper_color">
+                <color rgba="0.2 0.2 0.2 1.0"/>
+            </material>
+        </visual>
+    </link>
+    <joint name="gripper_mount_joint" type="fixed">
+        <parent link="wrist_link"/>
+        <child link="gripper_base_link"/>
+        <origin xyz="0 0 ${wrist_length}" rpy="0 0 0"/>
+    </joint>
+    <link name="left_finger_link">
+        <visual>
+            <origin xyz="0 0 ${finger_length/2}" rpy="0 0 0"/>
+            <geometry>
+                <box size="${finger_thickness} ${finger_width} ${finger_length}"/>
+            </geometry>
+            <material name="gripper_color"/>
+        </visual>
+    </link>
+    <joint name="left_finger_joint" type="prismatic">
+        <parent link="gripper_base_link"/>
+        <child link="left_finger_link"/>
+        <origin xyz="0 ${finger_gap} ${gripper_length}" rpy="0 0 0"/>
+        <axis xyz="0 1 0"/>
+        <limit lower="0" upper="0.02" effort="5" velocity="0.5"/>
+    </joint>
+    <link name="right_finger_link">
+        <visual>
+            <origin xyz="0 0 ${finger_length/2}" rpy="0 0 0"/>
+            <geometry>
+                <box size="${finger_thickness} ${finger_width} ${finger_length}"/>
+            </geometry>
+            <material name="gripper_color"/>
+        </visual>
+    </link>
+    <joint name="right_finger_joint" type="prismatic">
+        <parent link="gripper_base_link"/>
+        <child link="right_finger_link"/>
+        <origin xyz="0 -${finger_gap} ${gripper_length}" rpy="0 0 0"/>
+        <axis xyz="0 1 0"/>
+        <limit lower="-0.02" upper="0" effort="5" velocity="0.5"/>
+        <mimic joint="left_finger_joint" multiplier="-1" offset="0"/>
+    </joint>
 </robot>

Commit message: added lidar to the robot

File: src/robot_description/urdf/robot_description.urdf.xacro (robot description, xacro)
@@ -1,4 +1,5 @@
 <?xml version="1.0"?>
 <robot name="four_wheel_robot" xmlns:xacro="http://www.ros.org/wiki/xacro">
+    <xacro:arg name="mesh_path" default="package://robot_description/meshes/"/>
     <!-- mobile robot properties -->
     <xacro:property name="base_length" value="0.6"/>
@@ -231,3 +232,32 @@
         <mimic joint="left_finger_joint" multiplier="-1" offset="0"/>
     </joint>
+    <link name="lidar_link">
+        <visual>
+            <origin xyz="0 0 0" rpy="0 0 0"/>
+            <geometry>
+                <mesh filename="$(arg mesh_path)lidar.STL"/>
+            </geometry>
+            <material name="lidar_gray">
+                <color rgba="0.6 0.6 0.6 1.0"/>
+            </material>
+        </visual>
+        <collision>
+            <origin xyz="0 0 0" rpy="0 0 0"/>
+            <geometry>
+                <cylinder radius="0.06" length="0.04"/>
+            </geometry>
+        </collision>
+        <inertial>
+            <mass value="0.2"/>
+            <origin xyz="0 0 0" rpy="0 0 0"/>
+            <inertia ixx="0.0001" ixy="0.0" ixz="0.0"
+                    iyy="0.0001" iyz="0.0"
+                    izz="0.0001"/>
+        </inertial>
+    </link>
+    <joint name="lidar_joint" type="fixed">
+        <parent link="base_link"/>
+        <child link="lidar_link"/>
+        <origin xyz="0.28 0 ${base_height/2 + 0.02}" rpy="0 0 0"/>
+    </joint>
 </robot>

Commit message: added collision and inertial tags to the arm part

File: src/robot_description/urdf/robot_description.urdf.xacro (robot description, xacro)
@@ -14,5 +14,5 @@
     <xacro:property name="wheel_z_offset" value="-0.05"/>
     <!-- arm robot properties -->
-     <xacro:property name="link_radius" value="0.025"/>
+    <xacro:property name="link_radius" value="0.025"/>
     <xacro:property name="shoulder_length" value="0.05"/>
     <xacro:property name="upper_arm_length" value="0.15"/>
@@ -21,4 +21,11 @@
     <xacro:property name="gripper_length" value="0.05"/>
     <xacro:property name="finger_length" value="0.04"/>
+    <xacro:property name="arm_base_mass" value="0.1"/>
+    <xacro:property name="shoulder_mass" value="0.2"/>
+    <xacro:property name="upper_arm_mass" value="0.3"/>
+    <xacro:property name="forearm_mass" value="0.25"/>
+    <xacro:property name="wrist_mass" value="0.15"/>
+    <xacro:property name="gripper_base_mass" value="0.15"/>
+    <xacro:property name="finger_mass" value="0.05"/>
     <!-- gripper properties -->
      <xacro:property name="finger_width" value="0.015"/>
@@ -99,4 +106,28 @@
     <xacro:wheel prefix="rear_left"   x_reflect="-1" y_reflect="1"/>
     <xacro:wheel prefix="rear_right"  x_reflect="-1" y_reflect="-1"/>
+    <xacro:macro name="cylinder_inertial" params="mass radius length *origin">
+        <inertial>
+            <xacro:insert_block name="origin"/>
+            <mass value="${mass}"/>
+            <inertia
+                ixx="${(1/12) * mass * (3*radius*radius + length*length)}"
+                ixy="0.0" ixz="0.0"
+                iyy="${(1/12) * mass * (3*radius*radius + length*length)}"
+                iyz="0.0"
+                izz="${(1/2) * mass * radius*radius}"/>
+        </inertial>
+    </xacro:macro>
+    <xacro:macro name="box_inertial" params="mass x y z *origin">
+        <inertial>
+            <xacro:insert_block name="origin"/>
+            <mass value="${mass}"/>
+            <inertia
+                ixx="${(1/12) * mass * (y*y + z*z)}"
+                ixy="0.0" ixz="0.0"
+                iyy="${(1/12) * mass * (x*x + z*z)}"
+                iyz="0.0"
+                izz="${(1/12) * mass * (x*x + y*y)}"/>
+        </inertial>
+    </xacro:macro>
     <link name="arm_mount_link"/>
     <joint name="arm_mount_joint" type="fixed">
@@ -114,4 +145,12 @@
             </material>
         </visual>
+        <collision>
+            <geometry>
+                <cylinder radius="${link_radius*1.5}" length="${shoulder_length}"/>
+            </geometry>
+        </collision>
+        <xacro:cylinder_inertial mass="${arm_base_mass}" radius="${link_radius*1.5}" length="${shoulder_length}">
+            <origin xyz="0 0 0" rpy="0 0 0"/>
+        </xacro:cylinder_inertial>
     </link>
     <joint name="arm_base_joint" type="fixed">
@@ -127,4 +166,12 @@
             <material name="arm_color"/>
         </visual>
+        <collision>
+            <geometry>
+                <cylinder radius="${link_radius}" length="${shoulder_length}"/>
+            </geometry>
+        </collision>
+        <xacro:cylinder_inertial mass="${shoulder_mass}" radius="${link_radius}" length="${shoulder_length}">
+            <origin xyz="0 0 0" rpy="0 0 0"/>
+        </xacro:cylinder_inertial>
     </link>
     <joint name="shoulder_yaw_joint" type="revolute">
@@ -143,4 +190,13 @@
             <material name="arm_color"/>
         </visual>
+        <collision>
+            <origin xyz="0 0 ${upper_arm_length/2}" rpy="0 0 0"/>
+            <geometry>
+                <cylinder radius="${link_radius}" length="${upper_arm_length}"/>
+            </geometry>
+        </collision>
+        <xacro:cylinder_inertial mass="${upper_arm_mass}" radius="${link_radius}" length="${upper_arm_length}">
+            <origin xyz="0 0 ${upper_arm_length/2}" rpy="0 0 0"/>
+        </xacro:cylinder_inertial>
     </link>
     <joint name="shoulder_pitch_joint" type="revolute">
@@ -159,4 +215,13 @@
             <material name="arm_color"/>
         </visual>
+        <collision>
+            <origin xyz="0 0 ${forearm_length/2}" rpy="0 0 0"/>
+            <geometry>
+                <cylinder radius="${link_radius*0.8}" length="${forearm_length}"/>
+            </geometry>
+        </collision>
+        <xacro:cylinder_inertial mass="${forearm_mass}" radius="${link_radius*0.8}" length="${forearm_length}">
+            <origin xyz="0 0 ${forearm_length/2}" rpy="0 0 0"/>
+        </xacro:cylinder_inertial>
     </link>
     <joint name="elbow_pitch_joint" type="revolute">
@@ -175,4 +240,13 @@
             <material name="arm_color"/>
         </visual>
+        <collision>
+            <origin xyz="0 0 ${wrist_length/2}" rpy="0 0 0"/>
+            <geometry>
+                <cylinder radius="${link_radius*0.7}" length="${wrist_length}"/>
+            </geometry>
+        </collision>
+        <xacro:cylinder_inertial mass="${wrist_mass}" radius="${link_radius*0.7}" length="${wrist_length}">
+            <origin xyz="0 0 ${wrist_length/2}" rpy="0 0 0"/>
+        </xacro:cylinder_inertial>
     </link>
     <joint name="wrist_pitch_joint" type="revolute">
@@ -193,4 +267,13 @@
             </material>
         </visual>
+        <collision>
+            <origin xyz="0 0 ${gripper_length/2}" rpy="0 0 0"/>
+            <geometry>
+                <box size="0.05 0.06 ${gripper_length}"/>
+            </geometry>
+        </collision>
+        <xacro:box_inertial mass="${gripper_base_mass}" x="0.05" y="0.06" z="${gripper_length}">
+            <origin xyz="0 0 ${gripper_length/2}" rpy="0 0 0"/>
+        </xacro:box_inertial>
     </link>
     <joint name="gripper_mount_joint" type="fixed">
@@ -207,4 +290,13 @@
             <material name="gripper_color"/>
         </visual>
+        <collision>
+            <origin xyz="0 0 ${finger_length/2}" rpy="0 0 0"/>
+            <geometry>
+                <box size="${finger_thickness} ${finger_width} ${finger_length}"/>
+            </geometry>
+        </collision>
+        <xacro:box_inertial mass="${finger_mass}" x="${finger_thickness}" y="${finger_width}" z="${finger_length}">
+            <origin xyz="0 0 ${finger_length/2}" rpy="0 0 0"/>
+        </xacro:box_inertial>
     </link>
     <joint name="left_finger_joint" type="prismatic">
@@ -223,4 +315,13 @@
             <material name="gripper_color"/>
         </visual>
+        <collision>
+            <origin xyz="0 0 ${finger_length/2}" rpy="0 0 0"/>
+            <geometry>
+                <box size="${finger_thickness} ${finger_width} ${finger_length}"/>
+            </geometry>
+        </collision>
+        <xacro:box_inertial mass="${finger_mass}" x="${finger_thickness}" y="${finger_width}" z="${finger_length}">
+            <origin xyz="0 0 ${finger_length/2}" rpy="0 0 0"/>
+        </xacro:box_inertial>
     </link>
     <joint name="right_finger_joint" type="prismatic">
