Commit message: added ros2 control to the arm part

File: src/robot_description/urdf/robot_ros2_control.xacro (robot description, xacro)
@@ -37,4 +37,43 @@
             <state_interface name="velocity"/>
         </joint>
+        <joint name="shoulder_yaw_joint">
+            <command_interface name="position">
+                <param name="min">-3.1416</param>
+                <param name="max">3.1416</param>
+            </command_interface>
+            <state_interface name="position"/>
+        </joint>
+        <joint name="shoulder_pitch_joint">
+            <command_interface name="position">
+                <param name="min">-1.5708</param>
+                <param name="max">1.5708</param>
+            </command_interface>
+            <state_interface name="position"/>
+        </joint>
+        <joint name="elbow_pitch_joint">
+            <command_interface name="position">
+                <param name="min">0.0</param>
+                <param name="max">2.618</param>
+            </command_interface>
+            <state_interface name="position"/>
+        </joint>
+        <joint name="wrist_pitch_joint">
+            <command_interface name="position">
+                <param name="min">-1.5708</param>
+                <param name="max">1.5708</param>
+            </command_interface>
+            <state_interface name="position"/>
+        </joint>
+        <joint name="left_finger_joint">
+            <command_interface name="position">
+                <param name="min">0.0</param>
+                <param name="max">0.02</param>
+            </command_interface>
+            <state_interface name="position"/>
+        </joint>
+        <joint name="right_finger_joint">
+            <param name="mimic">left_finger_joint</param>
+            <param name="multiplier">-1</param>
+        </joint>
     </ros2_control>
 </robot>
